Commit message: Added bunch of things, including mppi controller

File: dyros_robotics_suite/dyros_robot_controller/robot/husky_dual_fr3.urdf (robot description, URDF)
Before this commit: robot husky_robot, 35 links, 34 joints
Links:
- added link l_fr3_hand, mass 0.73; collision mesh filename=package://franka_description/meshes/robot_ee/franka_hand_wh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; visual mesh filename=package://franka_description/meshes/robot_ee/franka_hand_wh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
- added link l_fr3_leftfinger; collision box size=17.5e-3 15.2e-3 18.5e-3; collision box size=17.5e-3 7e-3 23.5e-3
- added link l_fr3_rightfinger; collision box size=17.5e-3 15.2e-3 18.5e-3; collision box size=17.5e-3 7e-3 23.5e-3
- added link l_hand_tcp
- added link r_fr3_hand, mass 0.73; collision mesh filename=package://franka_description/meshes/robot_ee/franka_hand_wh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; visual mesh filename=package://franka_description/meshes/robot_ee/franka_hand_wh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
- added link r_fr3_leftfinger; collision box size=17.5e-3 15.2e-3 18.5e-3; collision box size=17.5e-3 7e-3 23.5e-3
- added link r_fr3_rightfinger; collision box size=17.5e-3 15.2e-3 18.5e-3; collision box size=17.5e-3 7e-3 23.5e-3
- added link r_hand_tcp
Joints:
- added joint l_fr3_finger_joint1: type fixed, parent l_fr3_hand, child l_fr3_leftfinger, origin xyz=0 0 0.0584 rpy=0 0 0, axis 0 1 0, limit lower=0.0 upper=0.04 effort=100 velocity=0.2
- added joint l_fr3_finger_joint2: type fixed, parent l_fr3_hand, child l_fr3_rightfinger, origin xyz=0 0 0.0584 rpy=0 0 0, axis 0 -1 0, limit lower=0.0 upper=0.04 effort=100 velocity=0.2, mimic joint=l_fr3_finger_joint1
- added joint l_fr3_hand_joint: type fixed, parent l_fr3_link8, child l_fr3_hand, origin xyz=0 0 0 rpy=0 0 -0.7853981633974483
- added joint l_hand_tcp_joint: type fixed, parent l_fr3_hand, child l_hand_tcp, origin xyz=0 0 0.1034 rpy=0 0 0
- added joint r_fr3_finger_joint1: type fixed, parent r_fr3_hand, child r_fr3_leftfinger, origin xyz=0 0 0.0584 rpy=0 0 0, axis 0 1 0, limit lower=0.0 upper=0.04 effort=100 velocity=0.2
- added joint r_fr3_finger_joint2: type fixed, parent r_fr3_hand, child r_fr3_rightfinger, origin xyz=0 0 0.0584 rpy=0 0 0, axis 0 -1 0, limit lower=0.0 upper=0.04 effort=100 velocity=0.2, mimic joint=r_fr3_finger_joint1
- added joint r_fr3_hand_joint: type fixed, parent r_fr3_link8, child r_fr3_hand, origin xyz=0 0 0 rpy=0 0 -0.7853981633974483
- added joint r_hand_tcp_joint: type fixed, parent r_fr3_hand, child r_hand_tcp, origin xyz=0 0 0.1034 rpy=0 0 0

File: dyros_robotics_suite/dyros_robot_controller/robot/husky_dual_fr3_vis.urdf (robot description, URDF)
Before this commit: robot husky_robot, 37 links, 36 joints
Links:
- added link l_fr3_hand, mass 0.73; collision mesh filename=package://franka_description/meshes/robot_ee/franka_hand_wh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; visual mesh filename=package://franka_description/meshes/robot_ee/franka_hand_wh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
- added link l_fr3_leftfinger; collision box size=17.5e-3 15.2e-3 18.5e-3; collision box size=17.5e-3 7e-3 23.5e-3
- added link l_fr3_rightfinger; collision box size=17.5e-3 15.2e-3 18.5e-3; collision box size=17.5e-3 7e-3 23.5e-3
- added link l_hand_tcp
- added link r_fr3_hand, mass 0.73; collision mesh filename=package://franka_description/meshes/robot_ee/franka_hand_wh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; visual mesh filename=package://franka_description/meshes/robot_ee/franka_hand_wh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
- added link r_fr3_leftfinger; collision box size=17.5e-3 15.2e-3 18.5e-3; collision box size=17.5e-3 7e-3 23.5e-3
- added link r_fr3_rightfinger; collision box size=17.5e-3 15.2e-3 18.5e-3; collision box size=17.5e-3 7e-3 23.5e-3
- added link r_hand_tcp
Joints:
- added joint l_fr3_finger_joint1: type fixed, parent l_fr3_hand, child l_fr3_leftfinger, origin xyz=0 0 0.0584 rpy=0 0 0, axis 0 1 0, limit lower=0.0 upper=0.04 effort=100 velocity=0.2
- added joint l_fr3_finger_joint2: type fixed, parent l_fr3_hand, child l_fr3_rightfinger, origin xyz=0 0 0.0584 rpy=0 0 0, axis 0 -1 0, limit lower=0.0 upper=0.04 effort=100 velocity=0.2, mimic joint=l_fr3_finger_joint1
- added joint l_fr3_hand_joint: type fixed, parent l_fr3_link8, child l_fr3_hand, origin xyz=0 0 0 rpy=0 0 -0.7853981633974483
- added joint l_hand_tcp_joint: type fixed, parent l_fr3_hand, child l_hand_tcp, origin xyz=0 0 0.1034 rpy=0 0 0
- added joint r_fr3_finger_joint1: type fixed, parent r_fr3_hand, child r_fr3_leftfinger, origin xyz=0 0 0.0584 rpy=0 0 0, axis 0 1 0, limit lower=0.0 upper=0.04 effort=100 velocity=0.2
- added joint r_fr3_finger_joint2: type fixed, parent r_fr3_hand, child r_fr3_rightfinger, origin xyz=0 0 0.0584 rpy=0 0 0, axis 0 -1 0, limit lower=0.0 upper=0.04 effort=100 velocity=0.2, mimic joint=r_fr3_finger_joint1
- added joint r_fr3_hand_joint: type fixed, parent r_fr3_link8, child r_fr3_hand, origin xyz=0 0 0 rpy=0 0 -0.7853981633974483
- added joint r_hand_tcp_joint: type fixed, parent r_fr3_hand, child r_hand_tcp, origin xyz=0 0 0.1034 rpy=0 0 0
