Commit message: Fixed self collision avoidance

File: dyros_robotics_suite/dyros_robot_controller/robot/husky_fr3.urdf (robot description, URDF)
Before this commit: robot husky_fr3, 26 links, 25 joints
Links:
- link fr3_link0: geometry visual mesh filename=package://franka_description/meshes/robot_arms/fr3/visual/l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
- link fr3_link1: geometry visual mesh filename=package://franka_description/meshes/robot_arms/fr3/visual/l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
- link fr3_link2: geometry visual mesh filename=package://franka_description/meshes/robot_arms/fr3/visual/l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
- link fr3_link3: geometry visual mesh filename=package://franka_description/meshes/robot_arms/fr3/visual/l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
- link fr3_link4: geometry visual mesh filename=package://franka_description/meshes/robot_arms/fr3/visual/l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
- link fr3_link5: geometry visual mesh filename=package://franka_description/meshes/robot_arms/fr3/visual/l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
- link fr3_link6: geometry visual mesh filename=package://franka_description/meshes/robot_arms/fr3/visual/l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
- link fr3_link7: geometry collision cylinder length=0.2 radius=0.05; visual mesh filename=package://franka_description/meshes/robot_arms/fr3/visual/l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
- link front_left_wheel: geometry 
- link front_right_wheel: geometry 
- link top_plate_link: geometry visual mesh filename=package://husky_description/meshes/top_plate.dae

File: dyros_robotics_suite/dyros_robot_controller/robot/husky_fr3_vis.urdf (robot description, URDF)
Before this commit: robot husky_fr3, 30 links, 29 joints
Links:
- link fr3_link0: geometry visual mesh filename=package://franka_description/meshes/robot_arms/fr3/visual/l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
- link fr3_link1: geometry visual mesh filename=package://franka_description/meshes/robot_arms/fr3/visual/l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
- link fr3_link2: geometry visual mesh filename=package://franka_description/meshes/robot_arms/fr3/visual/l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
- link fr3_link3: geometry visual mesh filename=package://franka_description/meshes/robot_arms/fr3/visual/l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
- link fr3_link4: geometry visual mesh filename=package://franka_description/meshes/robot_arms/fr3/visual/l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
- link fr3_link5: geometry visual mesh filename=package://franka_description/meshes/robot_arms/fr3/visual/l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
- link fr3_link6: geometry visual mesh filename=package://franka_description/meshes/robot_arms/fr3/visual/l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
- link fr3_link7: geometry collision cylinder length=0.2 radius=0.05; visual mesh filename=package://franka_description/meshes/robot_arms/fr3/visual/l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
